File: Plytki/P03-R6-review/eda/LINKS.kicad_sch (KiCad schematic)
At the start: 4 parts

Commit message: P03 R6 (S1), etap 4: README, ODBIOR, MECHANIKA, QA; MPN K15 = posiadany kod
Co-Authored-By: Claude Opus 5.5 <noreply@anthropic.com>
Claude-Session: https://claude.ai/code/session_01WcZWLEJhzUpXnmq1q9qQYv
Parts:
- J_BP1, J_BP2, J_BP3: MPN IDC box header 2x10, 2.54 mm, right angle, Au (e.g. Ampheno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 -> IDC box header 2x10, 2.54 mm, right angle, Au (MPN to be se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

Commit message: P03 R6: poprawki schematu po PR #6, layout w toku; przekazanie na Ubuntu 24/7
Schemat (src/run_schematic.py PASS: ERC 0, 511/511, funkcje 53/53, mutacje 44/44,
J_BP 12/12 + proby 25/25): R43 100k, trzecia zyla 5V_SYS na J_BP2.17 (PFAIL_N 16,
ADC_RESET 18), wszystkie R i C w SMD 1206, kolki listew serwisowych wedlug
polozenia wezlow (odwolania w ODBIOR.md poprawione).

Layout (niedomkniety): rozmieszczenie, zablokowany tor 5 V 1,5 mm, lancuch
run_layout.py i skrypty kontroli/PDF (jeszcze nieuruchomione). Stan, wyniki
przebiegow routera i decyzje sporne: Plytki/P03-R6-review/STAN-PRAC.md.

Srodowisko komputera 24/7 z Ubuntu: docs/UBUNTU-24-7.md; pamiec w docs/pamiec-claude.

Co-Authored-By: Claude Opus 5.5 <noreply@anthropic.com>
Connections:
- net 5V_SYS: now also J_BP2.17 (Pin_17)
- net ADC_RESET: now also J_BP2.18 (Pin_18); no longer J_BP2.16 (Pin_16)
- net GND: no longer J_BP2.17 (Pin_17)
- net PFAIL_N: now also J_BP2.16 (Pin_16); no longer J_BP2.18 (Pin_18)
Other:
- note added: "5V_SYS (J_BP2.17, 19, 20) i 3V3_IO (J_BP3.5) przychodza z P02 R4 przez P12. P12 rozprowadza ADC_SCLK i ADC_DOUTA do P05, P06 i P07."
- note removed: "5V_SYS (J_BP2.19-20) i 3V3_IO (J_BP3.5) przychodza z P02 R4 przez P12. P12 rozprowadza ADC_SCLK i ADC_DOUTA do P05, P06 i P07."
