File: Plytki/P03-R6-review/eda/OUT.kicad_sch (KiCad schematic)
At the start: 21 parts, among them U21 74LVC125A, U22 74LVC125A, U23 74LVC125A

Commit message: P03 R6 (S1), etap 4: README, ODBIOR, MECHANIKA, QA; MPN K15 = posiadany kod
Co-Authored-By: Claude Opus 5.5 <noreply@anthropic.com>
Claude-Session: https://claude.ai/code/session_01WcZWLEJhzUpXnmq1q9qQYv
Parts:
- C10, C11, C9: MPN K104K15X7RF53H5 -> K104K15X7RF5TH5

Commit message: P03 R6: poprawki schematu po PR #6, layout w toku; przekazanie na Ubuntu 24/7
Schemat (src/run_schematic.py PASS: ERC 0, 511/511, funkcje 53/53, mutacje 44/44,
J_BP 12/12 + proby 25/25): R43 100k, trzecia zyla 5V_SYS na J_BP2.17 (PFAIL_N 16,
ADC_RESET 18), wszystkie R i C w SMD 1206, kolki listew serwisowych wedlug
polozenia wezlow (odwolania w ODBIOR.md poprawione).

Layout (niedomkniety): rozmieszczenie, zablokowany tor 5 V 1,5 mm, lancuch
run_layout.py i skrypty kontroli/PDF (jeszcze nieuruchomione). Stan, wyniki
przebiegow routera i decyzje sporne: Plytki/P03-R6-review/STAN-PRAC.md.

Srodowisko komputera 24/7 z Ubuntu: docs/UBUNTU-24-7.md; pamiec w docs/pamiec-claude.

Co-Authored-By: Claude Opus 5.5 <noreply@anthropic.com>
Parts:
- C10, C11, C9: value 100nF / X7R -> 100nF / 50V X7R; footprint P03:C_Vishay_K15_H5_P5 -> Capacitor_SMD:C_1206_3216Metric_Pad1.33x1.80mm_HandSolder; MPN K104K15X7RF5TH5 -> GRM31CR71H104KA01L
- R15, R16, R17, R18, R19, R20, R21, R22, R23, R24: value 10K / 1% -> 10K / 1% 1206; footprint Resistor_THT:R_Axial_DIN0207_L6.3mm_D2.5mm_P5.08mm_Vertical -> Resistor_SMD:R_1206_3216Metric_Pad1.30x1.75mm_HandSolder; MPN MF0207FTE-10K -> RC1206FR-0710KL
