File: Plytki/P05-R3-review/eda/DIG.kicad_sch (KiCad schematic)
At the start: 17 parts, among them U10 74LVC125AD, U11 74LVC125AD, U9 74LVC125AD

Commit message: P05 R3 (S1) etap 2: typy części — SMD 1206, posiadane THT z rejestru, SW1 JS202011AQN
Rezystory precyzyjne 1206 0,1 %: okno DAQ_OK (R3-R8) 10 ppm/K, dzielniki
kanałów 25 ppm/K. Z rejestru: 47k i 4,7k MF0207 na stojąco, MKT 10n/100n,
MKS2 1u, C0G 1n, logika i 1N4148. Wyjątki: R1 1 W leżący, C1, C12/C13 1210.
SW1: suwak kątowy C&K JS202011AQN (biegun B lustrzany względem 7201).
ERC 0, 464/464 pinów.

Co-Authored-By: Claude Opus 5.5 <noreply@anthropic.com>
Claude-Session: https://claude.ai/code/session_01PNjhiJP63vXoN5NGrWe8up
Parts:
- R13: footprint Resistor_THT:R_Axial_DIN0207_L6.3mm_D2.5mm_P10.16mm_Horizontal -> Resistor_THT:R_Axial_DIN0207_L6.3mm_D2.5mm_P5.08mm_Vertical; MPN metal film resistor 47K 1% -> MF0207FTE-47K (Yageo MF0207 1% 0.6W, owned, standing)
- R14, R15, R16, R17, R18, R19, R20, R21, R22, R23, R24: footprint Resistor_THT:R_Axial_DIN0207_L6.3mm_D2.5mm_P10.16mm_Horizontal -> Resistor_SMD:R_1206_3216Metric_Pad1.30x1.75mm_HandSolder; MPN metal film resistor 10K 1% -> RC1206FR-0710KL
- R26, R27: footprint Resistor_SMD:R_0805_2012Metric -> Resistor_SMD:R_1206_3216Metric_Pad1.30x1.75mm_HandSolder; MPN 0805 1% 0.125W 33R -> RC1206FR-0733RL
