File: Plytki/P06-R2-review/eda/P06.kicad_sch (KiCad schematic)
At the start: 19 parts, among them U2 MCP6022-I/P, U4 MCP1702-3302E/TO, U5 74LVC125AD, U6 74LVC125AD, U7 SN74HC08N

Commit message: P06 R2: szprychy 4 x 2 mm na polach J3/J4, C17 100 nF na 5VA przy J5 (decyzje użytkownika 2.10)
- route_critical.py: pola przewodów J3/J4 na szprychach (wylewki mocy: szprycha 2 mm, szczelina 0,5 mm), RSH1 pełne;
  wylewka ECU_P1 pod J4.1 dłuższa o 2,45 mm (czwarta szprycha)
- schemat: C17 100 nF 1206 5VA_P06 / GND przy J5 (uwaga F7 recenzji); C1 zostaje X7R
- trasowanie zatwierdzonej wersji odtworzone, planer dołożył połączenia C17 (szerokość klasy PWR 0,6 mm w planerze)
- run_layout.py: return_check.py odrzuca próby z za długim powrotem masy odsprzęgania
- kontrole PCB 34/34 (siła: szprychy i korytarz liczone od wypełnienia wokół pól), próby ujemne 37/37

Co-Authored-By: Claude Opus 5.5 <noreply@anthropic.com>
Parts:
- added C17: 100n, Capacitor_SMD:C_1206_3216Metric_Pad1.33x1.80mm_HandSolder, symbol P06:C
Connections:
- net 5VA_P06: now also C17.1
- net GND: now also C17.2
