File: Plytki/P06-R2-review/routing/prerouted.kicad_pcb (KiCad board)
At the start: 2 copper layers, 106.5 x 100 mm, 81 parts, among them J3 ISERIES, J4 SW1 A, J5 SW1 B, U1 INA240A2, U10 MCP1525-I/TO, U2 MCP6022-I/P, U3 MCP3201-BI/P, U4 MCP1702-3302E/TO, U5 74LVC125AD, U6 74LVC125AD, U7 SN74HC08N, U8 MCP120-300DI/TO, U9 MCP120-450DI/TO

Commit message: P06 R2: poprawki po niezależnej recenzji PCB (2.10) — nadruk 1,0/0,15 mm, masa pod U2/U3, powrót masy odsprzęgania
- F1: wszystkie napisy nadruku >= 1,0 mm / 0,15 mm (minimum JLCPCB), minimum w regułach DRC
- F2/F3: wnętrza U2/U3, pas między nimi i strefa pod dolnymi pinami U2 bez obcej miedzi (strefy routera);
  kondensatory odsprzęgające rozmieszczane według padu zasilania i padu masy; C2 pod U3 przy IN+/IN-;
  D1 niżej; R30 przy U9.2; R10 pod U5; przelotki GND przy kondensatorach (stitch.py --targeted) i
  tor masy z planera dla C12 (complete_routes.py --ties)
- nowa kontrola: droga po miedzi GND kondensator -> pin GND układu (src/gndpath.py); odrzucanie prób
  trasowania z kolizjami miedzi
- DRC 0/0/0 (3 x lib_footprint_mismatch przyjęte), kontrole PCB 34/34, próby ujemne 37/37

Co-Authored-By: Claude Opus 5.5 <noreply@anthropic.com>
Parts:
- C2, R10, R14: moved to B.Cu
- R7: moved to F.Cu
- moved R30 63.7 mm to (91.5, 56.3), turned to -90 degrees
- moved R14 10.2 mm to (89.0, 40.7), turned to -90 degrees
- moved C2 9.13 mm to (60.0, 30.9), turned to -90 degrees
- moved R12 7.88 mm to (72.9, 40.0), turned to -90 degrees
- moved C6 7.74 mm to (41.2, 29.6), turned to -90 degrees
- moved C4 7.61 mm to (64.5, 44.8), turned to 180 degrees
- moved C11 7.27 mm to (94.0, 39.5), turned to 180 degrees
- moved R10 7.05 mm to (75.5, 28.5)
- moved R38 6.59 mm to (70.6, 31.1), turned to -90 degrees
- moved R9 6.15 mm to (68.7, 24.8)
- moved R7 5.74 mm to (68.7, 36.4), turned to 180 degrees
- moved C13 5.56 mm to (96.8, 45.1), turned to -90 degrees
- moved C10 5.51 mm to (78.0, 34.0), turned to 180 degrees
- moved C9 4.90 mm to (69.8, 41.3), turned to -90 degrees
- moved C1 4.63 mm to (42.0, 35.1), turned to -90 degrees
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Routing:
- net GND: track 92.5 -> 94.0 mm, vias 7 -> 8

Commit message: P06 R2: szprychy 4 x 2 mm na polach J3/J4, C17 100 nF na 5VA przy J5 (decyzje użytkownika 2.10)
- route_critical.py: pola przewodów J3/J4 na szprychach (wylewki mocy: szprycha 2 mm, szczelina 0,5 mm), RSH1 pełne;
  wylewka ECU_P1 pod J4.1 dłuższa o 2,45 mm (czwarta szprycha)
- schemat: C17 100 nF 1206 5VA_P06 / GND przy J5 (uwaga F7 recenzji); C1 zostaje X7R
- trasowanie zatwierdzonej wersji odtworzone, planer dołożył połączenia C17 (szerokość klasy PWR 0,6 mm w planerze)
- run_layout.py: return_check.py odrzuca próby z za długim powrotem masy odsprzęgania
- kontrole PCB 34/34 (siła: szprychy i korytarz liczone od wypełnienia wokół pól), próby ujemne 37/37

Co-Authored-By: Claude Opus 5.5 <noreply@anthropic.com>
Parts:
- added C17: 100n, Capacitor_SMD:C_1206_3216Metric_Pad1.33x1.80mm_HandSolder, F.Cu at (18.5, 69.9)
