File: Plytki/P06-R2-review/verification/negative-controls/return_cut/P06.kicad_pcb (KiCad board)
At the start: 2 copper layers, 106.5 x 100 mm, 81 parts, among them J3 ISERIES, J4 SW1 A, J5 SW1 B, U1 INA240A2, U10 MCP1525-I/TO, U2 MCP6022-I/P, U3 MCP3201-BI/P, U4 MCP1702-3302E/TO, U5 74LVC125AD, U6 74LVC125AD, U7 SN74HC08N, U8 MCP120-300DI/TO, U9 MCP120-450DI/TO

Commit message: P06 R2: szprychy 4 x 2 mm na polach J3/J4, C17 100 nF na 5VA przy J5 (decyzje użytkownika 2.10)
- route_critical.py: pola przewodów J3/J4 na szprychach (wylewki mocy: szprycha 2 mm, szczelina 0,5 mm), RSH1 pełne;
  wylewka ECU_P1 pod J4.1 dłuższa o 2,45 mm (czwarta szprycha)
- schemat: C17 100 nF 1206 5VA_P06 / GND przy J5 (uwaga F7 recenzji); C1 zostaje X7R
- trasowanie zatwierdzonej wersji odtworzone, planer dołożył połączenia C17 (szerokość klasy PWR 0,6 mm w planerze)
- run_layout.py: return_check.py odrzuca próby z za długim powrotem masy odsprzęgania
- kontrole PCB 34/34 (siła: szprychy i korytarz liczone od wypełnienia wokół pól), próby ujemne 37/37

Co-Authored-By: Claude Opus 5.5 <noreply@anthropic.com>
Parts:
- added C17: 100n, Capacitor_SMD:C_1206_3216Metric_Pad1.33x1.80mm_HandSolder, F.Cu at (18.5, 69.9)
Routing:
- net 5VA_P06: track 191.4 -> 210.8 mm, vias 2 -> 3
- net GND: vias 66 -> 67
