File: Plytki/P05-R3-review/routing/prerouted.kicad_pcb (KiCad board)
At the start: 2 copper layers, 106.5 x 100 mm, 127 parts, among them J4 TAPS / PTH, J6 AUX / coax 50mm, K1 G6K-2P-Y DC5, K2 G6K-2P-Y DC5, K3 G6K-2P-Y DC5, SW1 AUX HI / LO, U1 AD7606BBSTZ, U10 74LVC125AD, U11 74LVC125AD, U12 MCP1700-3302E/TO, U2 REF5025IDR, U3 TLV1702-Q1, U4 TBD62083APG, U5 SN74HC08N, U6 MCP120-300DI/TO, U7 MCP120-450DI/TO, U8 74LVC125AD, U9 74LVC125AD

Commit message: P05 R3: poprawki po niezależnej recenzji PCB (2.10) — masa przy U1, drogi powrotne, nadruk 1,0/0,15 mm
- MAJOR-1: bez paska 5VA (y 45) i kręgosłupa pod pinami wejść; łączniki 5VA pionowo między kondensatorami,
  AVCC 1 kręgosłupem wewnątrz pierścienia; przelotki GND pod korpusami kondensatorów, przy AGND/REFGND,
  pod każdym 100 nF, kolumna przy pinach wejść; 12 przelotek wewnątrz pierścienia (było 4)
- MAJOR-2: strefy routera na B.Cu pod wachlarzem wejść i kondensatorami U1; kondensatory odsprzęgające
  według pinu zasilania i GND; przelotki GND przy kondensatorach; tory masy z planera (C15, C18)
- MINOR: reguła 0,15 mm dla wylewek tylko w pierścieniu pól (obszary DRC_ONLY_*), VBAT >= 0,6 mm od TAP,
  rzeczywiste długości SPI w README, nadruk 1,0/0,15 mm, tabliczka P05-R3
- nowe kontrole dróg powrotnych masy (src/gndpath.py); dziewięć pozycji przyjętych jawnie (decyzja 1
  użytkownika 2.10, limity = zmierzone + ok. 1 mm)
- DRC 0/0/0 (4 x lib_footprint_mismatch przyjęte), kontrole PCB 36/36, próby ujemne 35/35

Co-Authored-By: Claude Opus 5.5 <noreply@anthropic.com>
Parts:
- moved R11 12.0 mm to (96.8, 77.5), turned to 0 degrees
- moved C17 9.67 mm to (83.1, 77.5), turned to 0 degrees
- moved C3 8.01 mm to (63.5, 23.0), turned to 180 degrees
- moved C20 7.27 mm to (78.5, 44.0), turned to -90 degrees
- moved C21 7.27 mm to (88.5, 27.0), turned to -90 degrees
- moved C18 7.25 mm to (97.8, 82.1)
- moved R22 7.02 mm to (82.8, 45.0), turned to 0 degrees
- moved R2 6.17 mm to (70.1, 27.5), turned to 0 degrees
- moved R45 6.10 mm to (76.2, 45.0), turned to 90 degrees
- moved R19 5.70 mm to (79.8, 51.8), turned to 0 degrees
- moved R16 5.46 mm to (78.5, 38.4), turned to 90 degrees
- moved R46 5.10 mm to (71.9, 43.7), turned to 180 degrees
- moved R23 4.58 mm to (82.1, 21.7), turned to 0 degrees
- moved C16 4.35 mm to (98.4, 54.1), turned to -90 degrees
- moved C22 3.10 mm to (78.5, 56.0), turned to -90 degrees
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Routing:
- net 3V3_DAQ: track 36.1 -> 28.5 mm
- net GND: track 222.7 -> 228.2 mm, vias 23 -> 33
- net 5VA_P05: track 45.9 -> 44.6 mm, vias 3 -> 4

Commit message: P05 R3: nóżki SW1 na GND, C35 10 µF na AVCC przy U1 (decyzje użytkownika 2.10)
- footprint ESW_100DP_M6: nóżki mocujące jako pola pinu 4 (GND) — oprawa przełącznika na masie (ESD)
- schemat: C35 10 µF 1206 X7R na 5VA_P05 nad C6 (uwaga recenzji o pojemności AVCC przy U1)
- trasowanie zatwierdzonej wersji odtworzone (C35 w miejscu wolnym od miedzi); planer z szerokością PWR 0,6 mm
- kontrole PCB 36/36, próby ujemne 35/35

Co-Authored-By: Claude Opus 5.5 <noreply@anthropic.com>
Parts:
- added C35: 10u, Capacitor_SMD:C_1206_3216Metric_Pad1.33x1.80mm_HandSolder, F.Cu at (57.3, 35.0)
