File: Plytki/P05-R3-review/verification/negative-controls/fan_track/P05.kicad_pcb (KiCad board)
At the start: 2 copper layers, 106.5 x 100 mm, 127 parts, among them J4 TAPS / PTH, J6 AUX / coax 50mm, K1 G6K-2P-Y DC5, K2 G6K-2P-Y DC5, K3 G6K-2P-Y DC5, SW1 AUX HI / LO, U1 AD7606BBSTZ, U10 74LVC125AD, U11 74LVC125AD, U12 MCP1700-3302E/TO, U2 REF5025IDR, U3 TLV1702-Q1, U4 TBD62083APG, U5 SN74HC08N, U6 MCP120-300DI/TO, U7 MCP120-450DI/TO, U8 74LVC125AD, U9 74LVC125AD

Commit message: P05 R3: nóżki SW1 na GND, C35 10 µF na AVCC przy U1 (decyzje użytkownika 2.10)
- footprint ESW_100DP_M6: nóżki mocujące jako pola pinu 4 (GND) — oprawa przełącznika na masie (ESD)
- schemat: C35 10 µF 1206 X7R na 5VA_P05 nad C6 (uwaga recenzji o pojemności AVCC przy U1)
- trasowanie zatwierdzonej wersji odtworzone (C35 w miejscu wolnym od miedzi); planer z szerokością PWR 0,6 mm
- kontrole PCB 36/36, próby ujemne 35/35

Co-Authored-By: Claude Opus 5.5 <noreply@anthropic.com>
Parts:
- added C35: 10u, Capacitor_SMD:C_1206_3216Metric_Pad1.33x1.80mm_HandSolder, F.Cu at (57.3, 35.0)
Routing:
- net GND: track 363.1 -> 360.8 mm, vias 104 -> 103
