File: Plytki/P11-R2-review/eda/CONTACTS.kicad_sch (KiCad schematic)
At the start: 10 parts, among them J11 CONTACTS, J8 TEST signal, X11 ARM momentary NO, X12 L1 detector 2NC, X13 L2 detector 2NC, X14 MARK momentary NO, X15 KEY TEST NO, X16 STOP latched NC+NO, X17 TEST detector NO, X8 TEST port AT04-12 key C

Commit message: P11 R2: decyzje użytkownika 4.10 i poprawki z recenzji
- klucze portów jak w R1: L1 = B, L2 = C, TEST = A (parts.py, BOM, PORTY.csv, schemat, README)
- prąd silnika port -> P06 / P07: 2,0 mm² (AWG14) na całej długości, styki złocone AT60-215-1631 / AT62-209-1631
- TAPy: mostki przy portach, jedna wiązka 5 par do P05 J4, masa komory 12 do GND J4 (przyjęte)
- J_P12: piny 12/18 GND; IDC 2x10 kątowe (Horizontal) na krawędzi P11 od strony ściany A
- notatka o stykach złoconych: odnośnik do verification/QA.md, prądy 0,31-0,32 mA (LOGGER) / do 0,87 mA (pełny)
- tabelka rysunkowa bez "PCB", komentarz w ramce; R1 z widocznym polem Wariant (LOGGER / DNP z P04)
- łańcuch run_schematic.py: ERC 0, 104/104 pinów, elektryczne 35/35 (mutacje 22/22), P12 22/22 (mutacje 13/13, próba zerowa czysta), manifest zgodny

Co-Authored-By: Claude Opus 5.5 <noreply@anthropic.com>
Parts:
- X8: value TEST port AT04-12 key C -> TEST port AT04-12 key A; MPN Amphenol AT04-12PC receptacle (pin contacts per data sheet;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 -> Amphenol AT04-12PA receptacle; cavities 1/2 (motor current)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
Other:
- note added: "Numery pinow X11...X17 sa FUNKCYJNE, nie katalogowe. P11-7: zwykle przyciski i przelaczniki ze stykami ZLOCONYMI, bez podswietlenia."
- note added: "Prad zamknietego styku: LOGGER ok. 0.31-0.32 mA, pelny 0.03-0.87 mA przy 3.3 V (verification/QA.md)."
- note removed: "Numery pinow X11...X17 sa FUNKCYJNE, nie katalogowe. P11-7: zwykle przyciski i przelaczniki ze stykami ZLOCONYMI (ok. 0.3 mA / 3.3 V), bez podswietlenia."
- company: Prototype / schematic + PCB review -> Prototype / schematic review - hardware not tested
