File: Plytki/P11-R2-review/eda/P11.kicad_sch (KiCad schematic)
At the start: 4 parts, among them J6 SCOPE tail, X6 SCOPE BNC

Commit message: P11 R2: decyzje użytkownika 4.10 i poprawki z recenzji
- klucze portów jak w R1: L1 = B, L2 = C, TEST = A (parts.py, BOM, PORTY.csv, schemat, README)
- prąd silnika port -> P06 / P07: 2,0 mm² (AWG14) na całej długości, styki złocone AT60-215-1631 / AT62-209-1631
- TAPy: mostki przy portach, jedna wiązka 5 par do P05 J4, masa komory 12 do GND J4 (przyjęte)
- J_P12: piny 12/18 GND; IDC 2x10 kątowe (Horizontal) na krawędzi P11 od strony ściany A
- notatka o stykach złoconych: odnośnik do verification/QA.md, prądy 0,31-0,32 mA (LOGGER) / do 0,87 mA (pełny)
- tabelka rysunkowa bez "PCB", komentarz w ramce; R1 z widocznym polem Wariant (LOGGER / DNP z P04)
- łańcuch run_schematic.py: ERC 0, 104/104 pinów, elektryczne 35/35 (mutacje 22/22), P12 22/22 (mutacje 13/13, próba zerowa czysta), manifest zgodny

Co-Authored-By: Claude Opus 5.5 <noreply@anthropic.com>
Parts:
- J_P12: value IDC 2x10 do P12 -> IDC 2x10 katowe do P12; footprint Connector_IDC:IDC-Header_2x10_P2.54mm_Vertical -> Connector_IDC:IDC-Header_2x10_P2.54mm_Horizontal; MPN Box header IDC 2x10 2.54 mm, gold (MPN in purchase task) -> Box header IDC 2x10 2.54 mm, right-angle, gold (MPN in purc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
- R1: Wariant (none) -> LOGGER: obsadzony / z P04: DNP
Other:
- note added: "J_P12: IDC 2x10 KATOWE do P12 (S1 8, PANELCORE + PANELSAFE), na krawedzi P11 od sciany A (P11 poziomo na dnie strefy panelu). Piny 10/13/14/15/16 jak P03 R6 J_BP1 (N_J_SCOPE_HOT, MARK, TEST_KEY, LOGGER_CLEAR, TEST_PRESENT)."
- note added: "Zwarcie PANEL_3V3-GND przy R1: 34 mA, 0.12 W w 1206 (0.25 W). Odbiorniki 3 x 10k do GND na P03 R6 (R27, R6, R8); MARK: 10k do 3V3_CORE na P03 R6."
- note removed: "J_P12: IDC 2x10 do P12 (S1 8, PANELCORE + PANELSAFE). Piny 10/13/14/15/16 jak P03 R6 J_BP1 (N_J_SCOPE_HOT, MARK, TEST_KEY, LOGGER_CLEAR, TEST_PRESENT)."
- note removed: "Zwarcie PANEL_3V3-GND przy R1: 33 mA, 0.11 W w 1206 (0.25 W). Odbiorniki 3 x 10k do GND na P03 R6 (R27, R6, R8); MARK: 10k do 3V3_CORE na P03 R6."
- company: Prototype / schematic + PCB review -> Prototype / schematic review - hardware not tested
