File: Plytki/M1-R1-review/eda/ADC.kicad_sch (KiCad schematic)
At the start: 35 parts, among them U3 AD7606BBSTZ

Commit message: M1 krok 6: PCB 150 x 80 mm, 4 warstwy, trasowanie zamkniete
DRC 0 / niepolaczone 0 / zgodnosc ze schematem 0, kontrole PCB 11/11,
proby ujemne 13/13. Tor 7,5 A jako wylewki F/B, para Kelvina zablokowana
(K_MINUS przez In2), miedz wokol AD7606B przeniesiona z P05 R3
(+37 / -15 mm). Lancuch z P07 S1, wydanie src/run_release.py.

Co-Authored-By: Claude Opus 5.5 <noreply@anthropic.com>
Parts:
- C14, C15: footprint Capacitor_SMD:C_1210_3225Metric_Pad1.33x2.70mm_HandSolder -> Capacitor_SMD:C_1210_3225Metric
