File: Plytki/M1-PCB-R1-zamowienie/projekt/routing/prerouted.kicad_pcb (KiCad board)
At the start: 4 copper layers, 150 x 80 mm, 97 parts, among them J1 BAT, J2 VMOTOR, J3 BTN, J4 IBT-2, J5 P1 ECU, J6 X1.7-16, M1 Waveshare ESP32-S3-DEV-KIT-N3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, U1 TSR 2-2450, U2 TSR 2-2433, U3 AD7606BBSTZ, U4 INA240A2, U5 74LVC125AD, U6 TCAN1051V, U7 74AHCT125D, U8 TPS2553DBVR

Commit message: M1-PCB-R1-zamowienie po recenzji: zrodlo z R2 4,7 k, ZIP 824058fb
Miedz bez zmian wzgledem poprzedniej wersji paczki (te same odcinki, przelotki,
wypelnienia); Gerbery roznia sie kolejnoscia apertur. CAM 24/24, proby ujemne
9/9 + zerowa, ogledziny nowych podgladow, FABRICATION_FILES_VERIFIED.

Co-Authored-By: Claude Opus 5.5 <noreply@anthropic.com>
Parts:
- R2: value 100K -> 4.7K
